Commit message: Added Gazebo files

File: src/scout_mini_description/urdf/scout_mini_gazebo.urdf.xacro (robot description, xacro)
@@ -23,4 +23,7 @@
         <cylinder radius="0.05" length="0.04"/>
       </geometry>
+      <material name="black">
+        <color rgba="0.1 0.1 0.1 1"/>
+      </material>
     </visual>
     <collision>
@@ -40,4 +43,5 @@
     <origin xyz="0.1 0 0.46" rpy="0 0 0"/>
   </joint>
+  <!-- Inertial link -->
   <joint name="inertial_joint" type="fixed">
     <parent link="base_link" />
@@ -52,4 +56,5 @@
     </inertial>
   </link>
+  <!-- Wheels -->
   <joint name="front_left_wheel_joint" type="continuous">
     <parent link="base_link" />
@@ -152,11 +157,8 @@
     </inertial>
   </link>
-  <!-- Hardware interface for REAL ROBOT -->
+  <!-- Gazebo-specific ros2_control -->
   <ros2_control name="scout_mini_control" type="system">
     <hardware>
-      <plugin>scout_mini_hardware/ScoutMiniHardware</plugin>
-      <param name="interface">can0</param>
-      <param name="wheel_radius">0.0875</param>
-      <param name="wheel_separation">0.490</param>
+      <plugin>gazebo_ros2_control/GazeboSystem</plugin>
     </hardware>
     <joint name="front_left_wheel_joint">
@@ -197,3 +199,83 @@
     </joint>
   </ros2_control>
+  <!-- Gazebo ros2_control plugin -->
+  <gazebo>
+    <plugin filename="libgazebo_ros2_control.so" name="gazebo_ros2_control">
+      <parameters>/apollo_ws/src/scout_mini_base/config/scout_mini.yaml</parameters>
+    </plugin>
+  </gazebo>
+  <!-- Gazebo LiDAR Plugin -->
+  <gazebo reference="laser_link">
+    <sensor name="lidar_sensor" type="ray">
+      <always_on>true</always_on>
+      <update_rate>10</update_rate>
+      <visualize>true</visualize>
+      <ray>
+        <scan>
+          <horizontal>
+            <samples>720</samples>
+            <resolution>1</resolution>
+            <min_angle>-3.14159</min_angle>
+            <max_angle>3.14159</max_angle>
+          </horizontal>
+        </scan>
+        <range>
+          <min>0.1</min>
+          <max>30.0</max>
+          <resolution>0.01</resolution>
+        </range>
+        <noise>
+          <type>gaussian</type>
+          <mean>0.0</mean>
+          <stddev>0.01</stddev>
+        </noise>
+      </ray>
+      <plugin name="gazebo_ros_laser_controller" filename="libgazebo_ros_ray_sensor.so">
+        <ros>
+          <namespace>/</namespace>
+          <remapping>~/out:=scan</remapping>
+        </ros>
+        <output_type>sensor_msgs/LaserScan</output_type>
+        <frame_name>laser_link</frame_name>
+      </plugin>
+    </sensor>
+  </gazebo>
+  <!-- Gazebo properties for better physics -->
+  <gazebo reference="base_link">
+    <material>Gazebo/Grey</material>
+    <mu1>0.2</mu1>
+    <mu2>0.2</mu2>
+  </gazebo>
+  <gazebo reference="front_left_wheel_link">
+    <material>Gazebo/Black</material>
+    <mu1>1.0</mu1>
+    <mu2>1.0</mu2>
+    <kp>1000000.0</kp>
+    <kd>100.0</kd>
+    <minDepth>0.001</minDepth>
+  </gazebo>
+  <gazebo reference="rear_left_wheel_link">
+    <material>Gazebo/Black</material>
+    <mu1>1.0</mu1>
+    <mu2>1.0</mu2>
+    <kp>1000000.0</kp>
+    <kd>100.0</kd>
+    <minDepth>0.001</minDepth>
+  </gazebo>
+  <gazebo reference="front_right_wheel_link">
+    <material>Gazebo/Black</material>
+    <mu1>1.0</mu1>
+    <mu2>1.0</mu2>
+    <kp>1000000.0</kp>
+    <kd>100.0</kd>
+    <minDepth>0.001</minDepth>
+  </gazebo>
+  <gazebo reference="rear_right_wheel_link">
+    <material>Gazebo/Black</material>
+    <mu1>1.0</mu1>
+    <mu2>1.0</mu2>
+    <kp>1000000.0</kp>
+    <kd>100.0</kd>
+    <minDepth>0.001</minDepth>
+  </gazebo>
 </robot>
